Commit message: Target: Include yoshi egg as model

File: kuka_arm/urdf/target.urdf.xacro (robot description, xacro)
@@ -7,8 +7,7 @@
     </inertial>
     <visual>
-      <origin xyz="0 0 0"/>
+      <origin xyz="-0.17 0.09 0"/>
       <geometry>
-        <cylinder radius="0.05" length="0.25"/>
-        <!--box size="0.10 0.10 0.25"/-->
+        <mesh filename="package://kuka_arm/models/yoshi_egg/yoshi_egg.dae" scale="0.02 0.02 0.02"/>
       </geometry>
     </visual>
@@ -22,5 +21,4 @@
   </link>
   <gazebo reference="target_link_1">
-    <material>Gazebo/Blue</material>
     <mu1>1.0</mu1>
     <mu2>1.0</mu2>
